File: ReceiverSampleBoard/ReceiverSampleBoard.kicad_pcb (KiCad board)
At the start: 2 copper layers, 11 parts, among them J1 Conn_01x02_Pin, Q1 IRLML0030, Q2 IRLML0030

Commit message: Traced Sample board
Parts:
- removed C1: C, Capacitor_SMD:C_1210_3225Metric
- moved J1 42.0 mm to (101.3, 118.0), turned to -90 degrees
- moved Q2 31.2 mm to (97.8, 82.0), turned to 180 degrees
- moved Q1 26.4 mm to (102.2, 82.0), turned to 0 degrees
- moved L5 24.1 mm to (112.5, 100.0), turned to 90 degrees
- moved L6 22.6 mm to (106.2, 89.2), turned to 150 degrees
- moved L2 22.1 mm to (87.5, 100.0), turned to -90 degrees
- moved L3 22.1 mm to (93.7, 110.8), turned to -30 degrees
- moved L1 21.7 mm to (93.7, 89.2), turned to -150 degrees
- moved L4 21.6 mm to (106.2, 110.8), turned to 30 degrees
- moved D1 16.9 mm to (100.0, 113.2), turned to 90 degrees
Routing:
- net GND: track 0.00 -> 119.3 mm
- net Net-(Q1-D): track 0.00 -> 67.6 mm
- net Net-(Q1-G): track 0.00 -> 61.7 mm
- net Net-(L3-Pad2): track 0.00 -> 9.47 mm
- net Net-(L1-Pad2): track 0.00 -> 7.84 mm
- net Net-(L4-Pad2): track 0.00 -> 7.84 mm
- net Net-(L2-Pad2): track 0.00 -> 7.84 mm
- net Net-(L5-Pad2): track 0.00 -> 7.84 mm
- net Net-(J1-Pin_1): track 0.00 -> 6.23 mm
Other:
- board outline added: 40 x 40 mm
