File: ReceiverSampleBoard/ReceiverSampleBoard.kicad_sch (KiCad schematic)
At the start: 11 parts, among them J1 Conn_01x02_Pin, Q1 IRLML0030, Q2 IRLML0030

Commit message: Traced Sample board
Parts:
- removed C1: C, Capacitor_SMD:C_1210_3225Metric, symbol Device:C
Other:
- moved on the sheet: J1
Changed lines of the file:
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@@
   (junction (at 152.4 92.71) (diameter 0) (color 0 0 0 0)
   )
-  (junction (at 177.8 97.79) (diameter 0) (color 0 0 0 0)
-  )
   (wire (pts (xy 152.4 106.68) (xy 152.4 107.95))
     (stroke (width 0) (type default))
@@
     (stroke (width 0) (type default))
   )
-  (wire (pts (xy 193.04 101.6) (xy 190.5 101.6))
+  (wire (pts (xy 180.34 101.6) (xy 177.8 101.6))
     (stroke (width 0) (type default))
   )
@@
     (stroke (width 0) (type default))
   )
-  (wire (pts (xy 193.04 104.14) (xy 190.5 104.14))
+  (wire (pts (xy 180.34 104.14) (xy 177.8 104.14))
     (stroke (width 0) (type default))
   )
@@
     (stroke (width 0) (type default))
   )
-  (wire (pts (xy 190.5 101.6) (xy 190.5 97.79))
-    (stroke (width 0) (type default))
-  )
-  (wire (pts (xy 177.8 97.79) (xy 177.8 99.06))
-    (stroke (width 0) (type default))
-  )
-  (wire (pts (xy 177.8 106.68) (xy 177.8 107.95))
+  (wire (pts (xy 177.8 69.85) (xy 177.8 101.6))
     (stroke (width 0) (type default))
   )
@@
     (stroke (width 0) (type default))
   )
-  (wire (pts (xy 190.5 104.14) (xy 190.5 107.95))
+  (wire (pts (xy 177.8 104.14) (xy 177.8 107.95))
     (stroke (width 0) (type default))
   )
@@
     (stroke (width 0) (type default))
   )
-  (wire (pts (xy 177.8 69.85) (xy 177.8 97.79))
-    (stroke (width 0) (type default))
-  )
   (wire (pts (xy 129.54 101.6) (xy 129.54 95.25))
     (stroke (width 0) (type default))
@@
     (stroke (width 0) (type default))
   )
-  (wire (pts (xy 190.5 97.79) (xy 177.8 97.79))
-    (stroke (width 0) (type default))
-  )
   (wire (pts (xy 101.6 90.17) (xy 101.6 95.25))
     (stroke (width 0) (type default))
@@
         (path "/cc913d1b-9400-4773-ba28-c10b3ba2aeb7"
           (reference "L4") (unit 1)
-        )
-      )
-    )
-  )
-  (symbol (lib_id "Device:C") (at 177.8 102.87 0) (unit 1)
-    (in_bom yes) (on_board yes) (dnp no) (fields_autoplaced)
-    (property "Reference" "C1" (at 181.61 101.6 0)
-      (effects (font (size 1.27 1.27)) (justify left))
-    )
-    (property "Value" "C" (at 181.61 104.14 0)
-      (effects (font (size 1.27 1.27)) (justify left))
-    )
-    (property "Footprint" "Capacitor_SMD:C_1210_3225Metric" (at 178.7652 106.68 0)
-      (effects (font (size 1.27 1.27)) hide)
-    )
-    (property "Datasheet" "~" (at 177.8 102.87 0)
-      (effects (font (size 1.27 1.27)) hide)
-    )
-    (pin "2")
-    (pin "1")
-    (instances
-      (project "ReceiverSampleBoard"
-        (path "/cc913d1b-9400-4773-ba28-c10b3ba2aeb7"
-          (reference "C1") (unit 1)
-        )
-      )
-    )
-  )
-  (symbol (lib_id "power:GND") (at 177.8 107.95 0) (unit 1)
-    (in_bom yes) (on_board yes) (dnp no) (fields_autoplaced)
-    (property "Reference" "#PWR03" (at 177.8 114.3 0)
-      (effects (font (size 1.27 1.27)) hide)
-    )
-    (property "Value" "GND" (at 177.8 113.03 0)
-      (effects (font (size 1.27 1.27)))
-    )
-    (property "Footprint" "" (at 177.8 107.95 0)
-      (effects (font (size 1.27 1.27)) hide)
-    )
-    (property "Datasheet" "" (at 177.8 107.95 0)
-      (effects (font (size 1.27 1.27)) hide)
-    )
-    (pin "1")
-    (instances
-      (project "ReceiverSampleBoard"
-        (path "/cc913d1b-9400-4773-ba28-c10b3ba2aeb7"
-          (reference "#PWR03") (unit 1)
         )
       )
@@
     )
   )
-  (symbol (lib_id "power:GND") (at 190.5 107.95 0) (unit 1)
-    (in_bom yes) (on_board yes) (dnp no) (fields_autoplaced)
-    (property "Reference" "#PWR04" (at 190.5 114.3 0)
-      (effects (font (size 1.27 1.27)) hide)
-    )
-    (property "Value" "GND" (at 190.5 113.03 0)
-      (effects (font (size 1.27 1.27)))
-    )
-    (property "Footprint" "" (at 190.5 107.95 0)
-      (effects (font (size 1.27 1.27)) hide)
-    )
-    (property "Datasheet" "" (at 190.5 107.95 0)
+  (symbol (lib_id "power:GND") (at 177.8 107.95 0) (unit 1)
+    (in_bom yes) (on_board yes) (dnp no) (fields_autoplaced)
+    (property "Reference" "#PWR04" (at 177.8 114.3 0)
+      (effects (font (size 1.27 1.27)) hide)
+    )
+    (property "Value" "GND" (at 177.8 113.03 0)
+      (effects (font (size 1.27 1.27)))
+    )
+    (property "Footprint" "" (at 177.8 107.95 0)
+      (effects (font (size 1.27 1.27)) hide)
+    )
+    (property "Datasheet" "" (at 177.8 107.95 0)
       (effects (font (size 1.27 1.27)) hide)
     )
@@
     )
   )
-  (symbol (lib_id "Connector:Conn_01x02_Pin") (at 198.12 101.6 0) (mirror y) (unit 1)
-    (in_bom yes) (on_board yes) (dnp no) (fields_autoplaced)
-    (property "Reference" "J1" (at 199.39 101.6 0)
+  (symbol (lib_id "Connector:Conn_01x02_Pin") (at 185.42 101.6 0) (mirror y) (unit 1)
+    (in_bom yes) (on_board yes) (dnp no) (fields_autoplaced)
+    (property "Reference" "J1" (at 186.69 101.6 0)
       (effects (font (size 1.27 1.27)) (justify right))
     )
-    (property "Value" "Conn_01x02_Pin" (at 199.39 104.14 0)
+    (property "Value" "Conn_01x02_Pin" (at 186.69 104.14 0)
       (effects (font (size 1.27 1.27)) (justify right))
     )
-    (property "Footprint" "Connector_PinHeader_2.54mm:PinHeader_1x02_P2.54mm_Horizontal" (at 198.12 101.6 0)
-      (effects (font (size 1.27 1.27)) hide)
-    )
-    (property "Datasheet" "~" (at 198.12 101.6 0)
-      (effects (font (size 1.27 1.27)) hide)
-    )
+    (property "Footprint" "Connector_PinHeader_2.54mm:PinHeader_1x02_P2.54mm_Horizontal" (at 185.42 101.6 0)
+      (effects (font (size 1.27 1.27)) hide)
+    )
+    (property "Datasheet" "~" (at 185.42 101.6 0)
+      (effects (font (size 1.27 1.27)) hide)
+    )
