File: Board/Tacho.kicad_pcb (KiCad board)
At the start: 2 copper layers, 40 x 40 mm, 31 parts, among them Q3 WST2007, U1 KTH1601, U2 PY32F002AW15U

Commit message: Updates to pcb
Parts:
- moved TP4 50.9 mm to (111.0, 119.0)
- moved TP1 48.8 mm to (111.0, 81.0)
- moved TP2 38.1 mm to (85.0, 125.0)
- moved TP3 33.5 mm to (89.0, 119.0)
- moved TP5 19.9 mm to (82.0, 100.0)
- moved R5 16.7 mm to (83.5, 92.8), turned to 90 degrees
- moved D5 4.12 mm to (100.0, 75.0), turned to 0 degrees
- moved R6 3.50 mm to (84.0, 114.0), turned to 180 degrees
- moved D4 3.04 mm to (100.0, 74.0), turned to 0 degrees
- moved D3 2.00 mm to (100.0, 73.0), turned to 0 degrees
- moved D2 1.12 mm to (100.0, 72.0), turned to 0 degrees
- moved D1 1.00 mm to (100.0, 71.0), turned to 0 degrees
Routing:
- net Net-(U2-PA4): track 0.00 -> 14.8 mm
- net Net-(U2-PA2): track 0.00 -> 7.30 mm
- net Net-(U2-PA3): track 0.00 -> 7.29 mm
- net Net-(U2-PF2-NRST): track 0.00 -> 4.00 mm
- net Net-(U2-PA1): track 0.00 -> 4.00 mm
- net Net-(U2-PA0): track 0.00 -> 4.00 mm
- net (no net): track 0.00 -> 4.00 mm
- net VCC: track 0.00 -> 2.88 mm
- net Net-(U1-OUTPUT): track 0.00 -> 1.55 mm

Commit message: Layout finished
Parts:
- removed U1: KTH1601, Package_TO_SOT_SMD:SOT-553
- added C5: 1uF, Capacitor_SMD:C_0402_1005Metric_Pad0.74x0.62mm_HandSolder, F.Cu at (96.0, 117.5)
- added R7: 10k, Resistor_SMD:R_0402_1005Metric, F.Cu at (97.0, 117.5)
- added U3: DRV5013, Package_TO_SOT_SMD:SOT-23, F.Cu at (100.0, 131.2)
- moved TP5 30.7 mm to (108.8, 84.8)
- moved TP2 25.1 mm to (82.5, 100.0)
- moved R1 25.1 mm to (85.5, 93.0), turned to 60 degrees
- moved R2 21.3 mm to (86.0, 90.8), turned to 60 degrees
- moved R3 20.2 mm to (84.2, 92.2), turned to 60 degrees
- moved TP1 20.1 mm to (117.5, 100.0)
- moved C1 19.1 mm to (103.0, 117.5), turned to -90 degrees
- moved C4 18.6 mm to (117.5, 95.0), turned to 90 degrees
- moved D6 17.4 mm to (115.2, 91.2), turned to 30 degrees
- moved R4 16.6 mm to (84.8, 90.0), turned to 60 degrees
- moved C2 9.52 mm to (112.2, 87.8), turned to 60 degrees
- moved C3 9.52 mm to (87.8, 112.2), turned to 60 degrees
- moved R6 9.12 mm to (82.5, 105.0), turned to -90 degrees
- moved TP3 4.45 mm to (91.2, 115.2)
- moved TP4 4.45 mm to (108.8, 115.2)
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Routing:
- net VCC: track 2.88 -> 128.2 mm, vias 0 -> 4
- net GND: track 0.00 -> 97.4 mm, vias 0 -> 6
- net Net-(U2-PA8): track 1.55 -> 34.9 mm
- net Net-(D5-K): track 0.00 -> 32.4 mm, vias 0 -> 2
- net Net-(D3-K): track 0.00 -> 30.6 mm
- net Net-(D4-K): track 0.00 -> 29.2 mm, vias 0 -> 2
- net Net-(D1-K): track 0.00 -> 28.0 mm
- net Net-(D2-K): track 0.00 -> 27.3 mm
- net Net-(U2-PA14-SWC): track 0.00 -> 25.5 mm, vias 0 -> 1
- net Net-(L4-Pad1): track 0.00 -> 19.2 mm, vias 0 -> 2
- net Net-(L3-Pad2): track 0.00 -> 19.2 mm, vias 0 -> 2
- net Net-(L5-Pad2): track 0.00 -> 19.2 mm, vias 0 -> 2
- net Net-(L2-Pad1): track 0.00 -> 19.2 mm, vias 0 -> 2
- net Net-(L1-Pad2): track 0.00 -> 19.2 mm, vias 0 -> 2
- net Net-(Q3A-G): track 0.00 -> 15.4 mm
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Other:
- board size 40 x 40 mm -> 40 x 62.8 mm
- board text added: "FZ 2024"

Commit message: Current limit and reset pullup resistors value changed
Parts:
- R1, R2, R3, R4, R5: value 30R -> 430R
- R6: value 4.7k -> 10k
Changed lines of the file:
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@@
         (effects (font (size 1 1) (thickness 0.15)))
     )
-    (fp_text value "30R" (at 0 1.17 60) (layer "F.Fab")
+    (fp_text value "430R" (at 0 1.17 60) (layer "F.Fab")
         (effects (font (size 1 1) (thickness 0.15)))
     )
@@
         (effects (font (size 1 1) (thickness 0.15)))
     )
-    (fp_text value "4.7k" (at 0 1.17 -270) (layer "F.Fab")
+    (fp_text value "10k" (at 0 1.17 -270) (layer "F.Fab")
         (effects (font (size 1 1) (thickness 0.15)))
     )
@@
         (effects (font (size 1 1) (thickness 0.15)))
     )
-    (fp_text value "30R" (at 0 1.17 60) (layer "F.Fab")
+    (fp_text value "430R" (at 0 1.17 60) (layer "F.Fab")
         (effects (font (size 1 1) (thickness 0.15)))
     )
@@
         (effects (font (size 1 1) (thickness 0.15)))
     )
-    (fp_text value "30R" (at 0 1.17 60) (layer "F.Fab")
+    (fp_text value "430R" (at 0 1.17 60) (layer "F.Fab")
         (effects (font (size 1 1) (thickness 0.15)))
     )
@@
         (effects (font (size 1 1) (thickness 0.15)))
     )
-    (fp_text value "30R" (at 0 1.17 60) (layer "F.Fab")
+    (fp_text value "430R" (at 0 1.17 60) (layer "F.Fab")
         (effects (font (size 1 1) (thickness 0.15)))
     )
@@
         (effects (font (size 1 1) (thickness 0.15)))
     )
-    (fp_text value "30R" (at 0 1.17 60) (layer "F.Fab")
-        (effects (font (size 1 1) (thickness 0.15)))
-    )
+    (fp_text value "430R" (at 0 1.17 60) (layer "F.Fab")
+        (effects (font (size 1 1) (thickness 0.15)))
+    )
